File: keyboard/keyboard.kicad_sch (KiCad schematic)
At the start: 200 parts

Commit message: Revert "Updated design for Kailh Choc V2 switches"
This reverts commit c061ce008c33d35abb33246c03603d5898ebf8bb.
Parts:
- S1, S10, S100, S11, S12, S13, S14, S15, S16, S17, S18, S19, S2, S20, S21, S22, S23, S24, S25, S26, S27, S28, S29, S3, S30, S31, S32, S34, S35, S36, S37, S39, S4, S40, S41, S42, S43, S44, S45, S46, S47, S48, S49, S5, S50, S52, S53, S54, S57, S58, S59, S6, S60, S61, S62, S63, S64, S65, S66, S67, S69, S7, S70, S71, S73, S74, S75, S76, S77, S78, S79, S8, S80, S81, S82, S84, S85, S86, S87, S9, S93, S94, S95, S96, S97, S98, S99: footprint ScottoKeebs_Hotswap:Hotswap_Choc_V2_1.00u -> ScottoKeebs_Hotswap:Hotswap_MX_1.00u
- S33: footprint ScottoKeebs_Hotswap:Hotswap_Choc_V2_2.00u -> ScottoKeebs_Hotswap:Hotswap_MX_2.00u
- S38, S51: footprint ScottoKeebs_Hotswap:Hotswap_Choc_V2_1.50u -> ScottoKeebs_Hotswap:Hotswap_MX_1.50u
- S55, S88: footprint ScottoKeebs_Hotswap:Hotswap_Choc_V2_2.00u_90deg -> ScottoKeebs_Hotswap:Hotswap_MX_2.00u_90deg
- S56, S83: footprint ScottoKeebs_Hotswap:Hotswap_Choc_V2_1.75u -> ScottoKeebs_Hotswap:Hotswap_MX_1.75u
- S68, S72: footprint ScottoKeebs_Hotswap:Hotswap_Choc_V2_2.25u -> ScottoKeebs_Hotswap:Hotswap_MX_2.25u
- S89, S90, S91: footprint ScottoKeebs_Hotswap:Hotswap_Choc_V2_1.25u -> ScottoKeebs_Hotswap:Hotswap_MX_1.25u
- S92: footprint ScottoKeebs_Hotswap:Hotswap_Choc_V2_6.25u -> ScottoKeebs_Hotswap:Hotswap_MX_6.25u

Commit message: Updated design for Kailh Choc V2 switches
Parts:
- S1, S10, S100, S11, S12, S13, S14, S15, S16, S17, S18, S19, S2, S20, S21, S22, S23, S24, S25, S26, S27, S28, S29, S3, S30, S31, S32, S34, S35, S36, S37, S39, S4, S40, S41, S42, S43, S44, S45, S46, S47, S48, S49, S5, S50, S52, S53, S54, S57, S58, S59, S6, S60, S61, S62, S63, S64, S65, S66, S67, S69, S7, S70, S71, S73, S74, S75, S76, S77, S78, S79, S8, S80, S81, S82, S84, S85, S86, S87, S9, S93, S94, S95, S96, S97, S98, S99: footprint ScottoKeebs_Hotswap:Hotswap_MX_1.00u -> ScottoKeebs_Hotswap:Hotswap_Choc_V2_1.00u
- S33: footprint ScottoKeebs_Hotswap:Hotswap_MX_2.00u -> ScottoKeebs_Hotswap:Hotswap_Choc_V2_2.00u
- S38, S51: footprint ScottoKeebs_Hotswap:Hotswap_MX_1.50u -> ScottoKeebs_Hotswap:Hotswap_Choc_V2_1.50u
- S55, S88: footprint ScottoKeebs_Hotswap:Hotswap_MX_2.00u_90deg -> ScottoKeebs_Hotswap:Hotswap_Choc_V2_2.00u_90deg
- S56, S83: footprint ScottoKeebs_Hotswap:Hotswap_MX_1.75u -> ScottoKeebs_Hotswap:Hotswap_Choc_V2_1.75u
- S68, S72: footprint ScottoKeebs_Hotswap:Hotswap_MX_2.25u -> ScottoKeebs_Hotswap:Hotswap_Choc_V2_2.25u
- S89, S90, S91: footprint ScottoKeebs_Hotswap:Hotswap_MX_1.25u -> ScottoKeebs_Hotswap:Hotswap_Choc_V2_1.25u
- S92: footprint ScottoKeebs_Hotswap:Hotswap_MX_6.25u -> ScottoKeebs_Hotswap:Hotswap_Choc_V2_6.25u
