File: keyboard/keyboard.kicad_pcb (KiCad board)
At the start: 2 copper layers, 380 x 150 mm, 209 parts, among them U1 Raspberry_Pi_Pico

Commit message: Updated the PCB design
Other:
- board size 380 x 150 mm -> 372 x 147.5 mm
Changed lines of the file:
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@@
 	(gr_poly
 		(pts
-			(xy 6.4 -13.1) (xy 6.4 136.9) (xy 386.4 136.9) (xy 386.4 -13.1) (xy 164.4 -13.1) (xy 164.4 -5.85)
-			(xy 212.9 -5.85) (xy 212.9 8.65) (xy 151.4 8.65) (xy 151.4 -13.1)
+			(xy 11.4 -13.1) (xy 11.4 134.4) (xy 383.4 134.4) (xy 383.4 -13.1) (xy 164.4 -13.1) (xy 164.4 -6.05)
+			(xy 212.9 -6.05) (xy 212.9 8.8) (xy 151.4 8.8) (xy 151.41 -13.1)
 		)
 		(stroke
